Commit message: Modified URDF to have create2

File: src/robot_hw/create_description/urdf/create_2.urdf.xacro (robot description, xacro)
@@ -2,5 +2,5 @@
 <robot name="create_2" xmlns:xacro="http://ros.org/wiki/xacro">
   <xacro:include filename="$(find create_description)/urdf/create_base.urdf.xacro" />
-  <xacro:include filename="$(find create_description)/urdf/create_2_gazebo.urdf.xacro" />
+  <!-- <xacro:include filename="$(find create_description)/urdf/create_2_gazebo.urdf.xacro" /> -->
   <xacro:create_base wheel_separation="0.235" base_diameter="0.3485">
     <mesh filename="package://create_description/meshes/create_2.dae" />

File: src/robot_hw/create_description/urdf/create_base.urdf.xacro (robot description, xacro)
@@ -65,4 +65,11 @@
     </collision>
     </link>
+    <link name="base_laser">
+    <inertial>
+      <mass value="0.01" />
+      <origin xyz="0 0 0" />
+      <inertia ixx="0.01" ixy="0.0" ixz="0.0" iyy="0.01" iyz="0.0" izz="0.5" />
+    </inertial>
+    </link>
     <link name="wall_sensor_link">
     <inertial>
@@ -129,4 +136,9 @@
       <parent link="base_link" />
       <child link="rightfront_cliff_sensor_link" />
+    </joint>
+    <joint name="base_link_base_laser_joint" type="fixed">
+      <origin xyz="0 0 0" rpy="0 0 0" />
+      <parent link="base_link" />
+      <child link="base_laser" />
     </joint>
     <xacro:create_wheel prefix="left" y_offset="${wheel_separation / 2}" wheel_radius="${wheel_radius}" wheel_width="${wheel_width}"/>
